Commit message: Fix camera topic nesting, add optical frame, fix odometry_source int type

File: src/amr_description/urdf/amr.urdf.xacro (robot description, xacro)
@@ -143,4 +143,161 @@
     <origin xyz="-0.25 0 0.05"/>
   </joint>
+    <!-- ========================= -->
+  <!-- 2D LIDAR -->
+  <!-- ========================= -->
+  <link name="laser_link">
+    <visual>
+      <geometry>
+        <cylinder radius="0.05" length="0.08"/>
+      </geometry>
+      <material name="gray"/>
+    </visual>
+    <collision>
+      <geometry>
+        <cylinder radius="0.05" length="0.08"/>
+      </geometry>
+    </collision>
+    <inertial>
+      <mass value="0.1"/>
+      <inertia
+        ixx="0.0001"
+        ixy="0.0"
+        ixz="0.0"
+        iyy="0.0001"
+        iyz="0.0"
+        izz="0.0001"/>
+    </inertial>
+  </link>
+  <joint name="laser_joint" type="fixed">
+    <parent link="base_link"/>
+    <child link="laser_link"/>
+    <!-- Mounted on top/front of robot -->
+    <origin xyz="0.15 0 0.30" rpy="0 0 0"/>
+  </joint>
+    <!-- ========================= -->
+  <!-- RGB CAMERA -->
+  <!-- ========================= -->
+  <link name="camera_link">
+    <visual>
+      <geometry>
+        <box size="0.08 0.06 0.05"/>
+      </geometry>
+      <material name="black"/>
+    </visual>
+    <collision>
+      <geometry>
+        <box size="0.08 0.06 0.05"/>
+      </geometry>
+    </collision>
+    <inertial>
+      <mass value="0.05"/>
+      <inertia
+        ixx="0.00001"
+        ixy="0.0"
+        ixz="0.0"
+        iyy="0.00001"
+        iyz="0.0"
+        izz="0.00001"/>
+    </inertial>
+  </link>
+  <joint name="camera_joint" type="fixed">
+    <parent link="base_link"/>
+    <child link="camera_link"/>
+    <!-- Front-facing camera -->
+    <origin xyz="0.30 0 0.25" rpy="0 0 0"/>
+  </joint>
+  <!-- ========================= -->
+  <!-- CAMERA OPTICAL FRAME -->
+  <!-- ========================= -->
+  <!-- FIX (item 3): gazebo_ros_camera publishes image/camera_info with the
+       frame_id set below in frame_name. camera_link itself follows URDF
+       convention (x-forward, z-up). ROS image/TF conventions expect an
+       "optical" frame (z-forward, x-right, y-down), or any pixel->3D
+       back-projection you do in Phase 4 will be rotated wrong. This adds
+       that frame as a zero-mass child and points frame_name at it below. -->
+  <link name="camera_optical_link"/>
+  <joint name="camera_optical_joint" type="fixed">
+    <parent link="camera_link"/>
+    <child link="camera_optical_link"/>
+    <origin xyz="0 0 0" rpy="-1.5708 0 -1.5708"/>
+  </joint>
+    <!-- ========================= -->
+<!-- GAZEBO RGB CAMERA SENSOR -->
+<!-- ========================= -->
+<gazebo reference="camera_link">
+  <sensor type="camera" name="camera1">
+    <always_on>true</always_on>
+    <update_rate>15.0</update_rate>
+    <visualize>false</visualize>
+    <camera name="head">
+      <horizontal_fov>1.047</horizontal_fov>
+      <image>
+        <width>640</width>
+        <height>480</height>
+        <format>R8G8B8</format>
+      </image>
+      <clip>
+        <near>0.1</near>
+        <far>20.0</far>
+      </clip>
+    </camera>
+   <plugin
+  name="camera_controller"
+  filename="libgazebo_ros_camera.so">
+  <!-- FIX (item 1): the old config set BOTH <namespace>camera</namespace>
+       AND <camera_name>camera_sensor</camera_name> while remapping
+       image_raw:=image_raw (a no-op, since source==target). Per the
+       gazebo_ros_camera docs, the published topic is built as
+       /<namespace>/<camera_name>/<remapped_name>, so that combination
+       was actually publishing to /camera/camera_sensor/image_raw, not the
+       /camera/image_raw you'd expect. Fix: drop <camera_name> and remap
+       to the full desired path instead, so the topic is exactly
+       /camera/image_raw and /camera/camera_info. Verify with:
+         ros2 topic list | grep camera -->
+  <ros>
+    <namespace>/</namespace>
+    <remapping>image_raw:=camera/image_raw</remapping>
+    <remapping>camera_info:=camera/camera_info</remapping>
+  </ros>
+  <!-- frame_name now points at the optical frame added above -->
+  <frame_name>camera_optical_link</frame_name>
+</plugin>
+  </sensor>
+</gazebo>
+    <!-- ========================= -->
+  <!-- GAZEBO RAY SENSOR -->
+  <!-- ========================= -->
+  <gazebo reference="laser_link">
+    <sensor name="laser_sensor" type="ray">
+      <always_on>true</always_on>
+      <visualize>true</visualize>
+      <update_rate>10.0</update_rate>
+      <ray>
+        <scan>
+          <horizontal>
+            <samples>360</samples>
+            <resolution>1</resolution>
+            <min_angle>-3.14159</min_angle>
+            <max_angle>3.14159</max_angle>
+          </horizontal>
+        </scan>
+        <range>
+          <min>0.12</min>
+          <max>10.0</max>
+          <resolution>0.01</resolution>
+        </range>
+      </ray>
+      <plugin
+        name="gazebo_ros_ray_sensor"
+        filename="libgazebo_ros_ray_sensor.so">
+        <ros>
+          <namespace>/</namespace>
+          <remapping>~/out:=scan</remapping>
+        </ros>
+        <output_type>sensor_msgs/LaserScan</output_type>
+        <frame_name>laser_link</frame_name>
+      </plugin>
+    </sensor>
+  </gazebo>
   <!-- ========================= -->
   <!-- GAZEBO PHYSICS -->
